File: Diagrama-Eduproto.sch (EAGLE design)
At the start: 31 parts, among them IC1 7805TV, Q1 4MHz

Commit message: new rev
Parts:
- removed U$2: TACTILE-SWITCH-PTH, GeekAmmo:TACTILE-SWITCH-PTH
- added R5: 47k, adafruit:R-US_0207/10
- added U$5: TACTILE-SWITCH-2P, GeekAmmo:TACTILE-SWITCH-2P
- C1, C2: device adafruit:CPOL-USE2.5-6 -> adafruit:CPOL-USE1.8-4
- C5: device adafruit:C-US075-042X103 -> adafruit:C-US050-025X075
- D1, D2: value (none) -> 1N4004; device SparkFun-DiscreteSemi:DIODEPTH -> adafruit:1N4004
- JP4, JP5: device adafruit:PINHD-1X6 -> adafruit:PINHD-1X6B
- JP6, JP7: device adafruit:PINHD-1X3 -> adafruit:PINHD-1X3CB
- S2: device switch:M9040P -> SparkFun-Switches:SWITCH-SPDT-PTH-11.6X4.0MM
Connections:
- removed net RXPLL: U$1.RC7/RX/DT/SDO, U$3.6
- new net RC7: R5.1, U$1.RC7/RX/DT/SDO, U$3.6
- net GND: now also U$5.3; no longer U$2.3, U$2.4
- net RESET: now also U$5.1; no longer U$2.1, U$2.2
- net VDD: now also R5.2
Other:
- moved on the sheet: C1, C2, C3, C4, C5, IC1, JP1, JP2, JP4, JP5, JP6, JP7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
