File: gerbers/Diagrama-Eduproto.brd (EAGLE design)
At the start: 99 x 46 mm, 32 parts, among them IC1 7805TV, Q1 4MHz

Commit message: new rev
Parts:
- C3, C4: device adafruit:C050-024X044 -> adafruit:C025-024X044
- moved C4 0.99 mm to (45.5, 35.0)
- moved C3 0.44 mm to (45.5, 39.6)
Routing:
- net OSC2: track 15.5 -> 16.7 mm
- net GND: track 255.7 -> 256.7 mm
Other:
- board text added: "2017"
- board text added: "CETI - 2017B - 6G"
- board text removed: "2018"
- board text removed: "CETI - 2018A"
Changed lines of the file:
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@@
 <setting verticaltext="up"/>
 </settings>
-<grid distance="0.01" unitdist="mm" unit="mm" style="lines" multiple="1" display="yes" altdistance="0.025" altunitdist="inch" altunit="inch"/>
+<grid distance="0.0025" unitdist="inch" unit="inch" style="lines" multiple="1" display="yes" altdistance="0.025" altunitdist="inch" altunit="inch"/>
 <layers>
 <layer number="1" name="Top" color="4" fill="1" visible="yes" active="yes"/>
@@
 <wire x1="99" y1="4" x2="99" y2="42" width="0" layer="20"/>
 <wire x1="95" y1="46" x2="4" y2="46" width="0" layer="20"/>
-<text x="42.7265" y="2.9565" size="1.778" layer="25" font="vector" ratio="10" distance="40">CETI - 2018A</text>
+<text x="42.7265" y="2.9565" size="1.778" layer="25" font="vector" ratio="10" distance="40">CETI - 2017B - 6G</text>
 <text x="46.25" y="9.5" size="1.6764" layer="25" font="vector" ratio="10" rot="R90">RD7</text>
 <text x="43.75" y="9.5" size="1.6764" layer="25" font="vector" ratio="10" rot="R90">RD6</text>
@@
 <vertex x="42.5" y="24"/>
 </polygon>
-<text x="9.9618375" y="37.902625" size="2.54" layer="22" font="vector" rot="SMR0">2018</text>
+<text x="9.9618375" y="37.902625" size="2.54" layer="22" font="vector" rot="SMR0">2017</text>
 <circle x="3.2" y="8.5" radius="1.8" width="0.254" layer="21"/>
 <text x="97.7198375" y="41.045125" size="1.6764" layer="22" font="vector" rot="SMR270">@Ware EduProto III - 4553</text>
@@
 <attribute name="VALUE" x="8.077" y="37.373" size="1.27" layer="27" font="vector" ratio="10"/>
 </element>
-<element name="C3" library="adafruit" package="C050-024X044" value="22pF" x="45.7" y="40" smashed="yes">
-<attribute name="VALUE" x="43.541" y="37.333" size="1.27" layer="27" font="vector" ratio="10"/>
-</element>
-<element name="C4" library="adafruit" package="C050-024X044" value="22pF" x="45.7" y="36" smashed="yes"/>
+<element name="C3" library="adafruit" package="C025-024X044" value="22pF" x="45.47" y="39.62" smashed="yes">
+<attribute name="VALUE" x="43.311" y="36.953" size="1.27" layer="27" font="vector" ratio="10"/>
+</element>
+<element name="C4" library="adafruit" package="C025-024X044" value="22pF" x="45.47" y="35.04" smashed="yes"/>
 <element name="C5" library="adafruit" package="C050-025X075" value="220nF" x="21.34" y="35.81" smashed="yes" rot="R180">
 <attribute name="VALUE" x="23.999" y="34.227" size="1.27" layer="27" font="vector" ratio="10" rot="R180"/>
@@
 <wire x1="55.63" y1="25.65" x2="53.09" y2="28.19" width="0.6096" layer="16"/>
 <wire x1="53.09" y1="28.19" x2="53.09" y2="30.73" width="0.6096" layer="16"/>
-<wire x1="53.09" y1="30.73" x2="53.09" y2="32.37" width="0.6096" layer="16"/>
-<wire x1="53.09" y1="32.37" x2="53.82" y2="33.1" width="0.6096" layer="16"/>
-<wire x1="53.82" y1="33.1" x2="54.6" y2="33.1" width="0.6096" layer="16"/>
-<wire x1="54.6" y1="33.1" x2="55.63" y2="34.13" width="0.6096" layer="16"/>
-<wire x1="55.63" y1="34.13" x2="55.63" y2="40.89" width="0.6096" layer="16"/>
+<wire x1="53.09" y1="30.73" x2="55.63" y2="33.27" width="0.6096" layer="16"/>
+<wire x1="55.63" y1="33.27" x2="55.63" y2="40.89" width="0.6096" layer="16"/>
 </signal>
 <signal name="TXLED">
@@
 <wire x1="70.87" y1="24.38" x2="54.36" y2="24.38" width="0.6096" layer="16"/>
 <wire x1="54.36" y1="24.38" x2="50.55" y2="28.19" width="0.6096" layer="16"/>
-<wire x1="50.55" y1="30.73" x2="50.55" y2="28.19" width="0.6096" layer="16"/>
-<wire x1="50.55" y1="40.89" x2="54.36" y2="37.08" width="0.6096" layer="16"/>
+<wire x1="50.55" y1="28.19" x2="50.55" y2="30.73" width="0.6096" layer="16"/>
+<wire x1="50.55" y1="30.73" x2="54.36" y2="34.54" width="0.6096" layer="16"/>
+<wire x1="54.36" y1="34.54" x2="54.36" y2="37.08" width="0.6096" layer="16"/>
+<wire x1="54.36" y1="37.08" x2="50.55" y2="40.89" width="0.6096" layer="16"/>
 <wire x1="50.55" y1="40.89" x2="49.28" y2="40.89" width="0.6096" layer="16"/>
 <wire x1="49.28" y1="40.89" x2="48.01" y2="42.16" width="0.6096" layer="16"/>
@@
 <wire x1="27.69" y1="40.89" x2="27.69" y2="42.16" width="0.6096" layer="16"/>
 <wire x1="27.69" y1="42.16" x2="28.96" y2="43.43" width="0.6096" layer="16"/>
-<wire x1="54.36" y1="37.08" x2="54.36" y2="35.05" width="0.6096" layer="16"/>
-<wire x1="54.36" y1="35.05" x2="52.88" y2="33.57" width="0.6096" layer="16"/>
-<wire x1="52.88" y1="33.57" x2="52.58" y2="33.57" width="0.6096" layer="16"/>
-<wire x1="50.55" y1="31.54" x2="50.55" y2="30.73" width="0.6096" layer="16"/>
-<wire x1="52.58" y1="33.57" x2="50.55" y2="31.54" width="0.6096" layer="16"/>
 </signal>
 <signal name="GND">
@@
 <wire x1="42.93" y1="30.73" x2="42.93" y2="32.18" width="0.6096" layer="16"/>
 <wire x1="42.93" y1="32.18" x2="43.75" y2="33" width="0.6096" layer="16"/>
+<wire x1="43.75" y1="33" x2="46" y2="33" width="0.6096" layer="16"/>
+<wire x1="46" y1="33" x2="46.75" y2="33.75" width="0.6096" layer="16"/>
+<wire x1="46.75" y1="33.75" x2="46.75" y2="35.03" width="0.6096" layer="16"/>
+<wire x1="46.75" y1="35.03" x2="46.74" y2="35.04" width="0.6096" layer="16"/>
+<wire x1="46.74" y1="35.5" x2="46.74" y2="35.04" width="0.6096" layer="16"/>
+<wire x1="46.74" y1="35.5" x2="46.74" y2="39.62" width="0.6096" layer="16"/>
+<wire x1="47.05" y1="35.81" x2="46.74" y2="35.5" width="0.6096" layer="16"/>
+<wire x1="52.84" y1="35.81" x2="47.05" y2="35.81" width="0.6096" layer="16"/>
 <polygon width="0.254" layer="1" isolate="0.4064">
 <vertex x="0" y="46"/>
@@
 <wire x1="83.76" y1="37.25" x2="83.76" y2="41.24" width="0.6096" layer="16"/>
 <wire x1="83.76" y1="41.24" x2="80.75" y2="44.25" width="0.6096" layer="16"/>
-<wire x1="48.24" y1="36" x2="48.24" y2="40" width="0.6096" layer="16"/>
-<wire x1="48.24" y1="36" x2="52.65" y2="36" width="0.6096" layer="16"/>
-<wire x1="52.65" y1="36" x2="52.84" y2="35.81" width="0.6096" layer="16"/>
-<wire x1="43.75" y1="33" x2="43.75" y2="33.01" width="0.6096" layer="16"/>
-<wire x1="43.75" y1="33.01" x2="44.31" y2="33.57" width="0.6096" layer="16"/>
-<wire x1="44.31" y1="33.57" x2="45.81" y2="33.57" width="0.6096" layer="16"/>
-<wire x1="45.81" y1="33.57" x2="48.24" y2="36" width="0.6096" layer="16"/>
 </signal>
 <signal name="N$11">
@@
 <contactref element="U$1" pad="13"/>
 <wire x1="40.39" y1="30.73" x2="40.39" y2="34.647" width="0.6096" layer="16"/>
-<wire x1="40.39" y1="34.647" x2="39.37" y2="35.667" width="0.6096" layer="16"/>
-<wire x1="39.37" y1="35.667" x2="42.827" y2="35.667" width="0.6096" layer="16"/>
-<wire x1="42.827" y1="35.667" x2="43.16" y2="36" width="0.6096" layer="16"/>
+<wire x1="40.0185" y1="35.0185" x2="40.39" y2="34.647" width="0.6096" layer="16"/>
+<wire x1="40.0185" y1="35.0185" x2="39.37" y2="35.667" width="0.6096" layer="16"/>
+<wire x1="44.2" y1="35.04" x2="40.04" y2="35.04" width="0.6096" layer="16"/>
+<wire x1="40.04" y1="35.04" x2="40.0185" y2="35.0185" width="0.6096" layer="16"/>
 </signal>
 <signal name="OSC2">
@@
 <wire x1="38" y1="33" x2="38" y2="30.88" width="0.6096" layer="16"/>
 <wire x1="38" y1="30.88" x2="37.85" y2="30.73" width="0.6096" layer="16"/>
-<wire x1="39.37" y1="40.493" x2="39.377" y2="40.5" width="0.6096" layer="16"/>
-<wire x1="42.66" y1="40.5" x2="43.16" y2="40" width="0.6096" layer="16"/>
-<wire x1="39.377" y1="40.5" x2="42.66" y2="40.5" width="0.6096" layer="16"/>
+<wire x1="44.2" y1="39.62" x2="41.88" y2="39.62" width="0.6096" layer="16"/>
+<wire x1="41.88" y1="39.62" x2="41" y2="40.5" width="0.6096" layer="16"/>
+<wire x1="41" y1="40.5" x2="39.377" y2="40.5" width="0.6096" layer="16"/>
+<wire x1="39.377" y1="40.5" x2="39.37" y2="40.493" width="0.6096" layer="16"/>
 </signal>
 <signal name="AUTORUN">
